File: ESP32_UniBoard.kicad_sch (KiCad schematic)
At the start: 30 parts, among them J1 USB_C_Receptacle_USB2.0, J2 Conn_01x06_Socket, J3 Hirose DF40C, SW1 SW_Push, SW2 SW_Push, U1 ESP32-S3-WROOM-1, U2 AZ1117-3.3, U3 USBLC6-2SC6

Commit message: Slight changes and added JLCPCB part numbers
Parts:
- C1: JLCPCB Part # (none) -> C15849
- C2, C4, C5, C9: JLCPCB Part # (none) -> C14663
- C3, C8: JLCPCB Part # (none) -> C19702
- C6: JLCPCB Part # (none) -> C59461
- D1: value D_Schottky -> B5819W SL; footprint Diode_SMD:D_0603_1608Metric -> Diode_SMD:D_SOD-123; JLCPCB Part # (none) -> C8598
- D2: JLCPCB Part # (none) -> C2833058
- D3: value RED -> YL; JLCPCB Part # (none) -> C131265
- D4: JLCPCB Part # (none) -> C131265
- F1: value Polyfuse -> 1.1 A; JLCPCB Part # (none) -> C207024
- J1: JLCPCB Part # (none) -> C2988369
- J3: value Hirose DF40C -> dHirose DF40C-50DS; JLCPCB Part # (none) -> C424646
- R1, R2: JLCPCB Part # (none) -> C144594
- R3: JLCPCB Part # (none) -> C116677
- R4: value R -> 680R; JLCPCB Part # (none) -> C115415
- R5, R6: value R -> 1k8; JLCPCB Part # (none) -> C228145
- SW1, SW2: JLCPCB Part # (none) -> C354943
- U1: JLCPCB Part # (none) -> C2913198
- U3: JLCPCB Part # (none) -> C5261088
Other:
- company: (none) -> D. Frei
- title: (none) -> ESP32 UniBoard
